Commit message: add

File: ros2_ws/src/xe_tham_do/description/camera.xacro (robot description, xacro)
@@ -1,22 +1,4 @@
 <?xml version="1.0"?>
 <robot xmlns:xacro="http://www.ros.org/wiki/xacro" >
-    <!--
-        File này định nghĩa cảm biến camera trong mô hình robot sử dụng URDF/xacro.
-        - <joint> "camera_joint" liên kết cố định giữa thân xe (chassis) và khung camera (camera_link).
-        - <link> "camera_link" mô tả hình học của camera:
-            + Bao gồm một hình hộp (box) để mô phỏng thân camera.
-            + Một hình trụ nhỏ (cylinder) để mô phỏng ống kính hoặc giá đỡ.
-        - <joint> "camera_optical_joint" liên kết cố định từ "camera_link" tới "camera_link_optical", dùng để thiết lập hệ trục quang học đúng chuẩn của camera.
-        - <link> "camera_link_optical" là frame gắn với dữ liệu hình ảnh xuất ra.
-        - <gazebo> cấu hình cảm biến camera trong mô phỏng Gazebo:
-            + Gắn vật liệu màu đen cho camera.
-            + Khai báo cảm biến loại "camera" với các tham số:
-                * Góc nhìn ngang (horizontal_fov): 1.089 rad.
-                * Kích thước ảnh: 640x480, định dạng màu R8G8B8.
-                * Cận clip: 0.05m, xa clip: 8m.
-                * Tần số cập nhật: 10Hz.
-            + Plugin "camera_controller" xuất dữ liệu hình ảnh với frame_name là "camera_link_optical".
-        File này giúp tích hợp camera cho robot cả trên mô phỏng (Gazebo) lẫn thực tế (ROS).
-    -->
     <joint name="camera_joint" type="fixed">
         <parent link="chassis"/>

File: ros2_ws/src/xe_tham_do/description/inertial_macros.xacro (robot description, xacro)
@@ -1,14 +1,4 @@
 <?xml version="1.0"?>
 <robot xmlns:xacro="http://www.ros.org/wiki/xacro" >
-    <!--
-        File này chứa các macro xacro để tính toán quán tính cho các hình học cơ bản trong robot (hình cầu, hộp, trụ).
-        Các macro này giúp bạn dễ dàng khai báo khối lượng và ma trận quán tính cho các liên kết trong mô hình URDF.
-        - inertial_sphere: Tính quán tính cho hình cầu.
-        - inertial_box: Tính quán tính cho hình hộp chữ nhật.
-        - inertial_cylinder: Tính quán tính cho hình trụ.
-        Công thức tham khảo từ: https://en.wikipedia.org/wiki/List_of_moments_of_inertia
-        Bạn có thể sử dụng các macro này để khai báo thuộc tính <inertial> cho từng link trong robot.
-        Tham số *origin cho phép bạn truyền vào thuộc tính origin nếu cần.
-    -->
     <!-- Specify some standard inertial calculations https://en.wikipedia.org/wiki/List_of_moments_of_inertia -->
     <!-- These make use of xacro's mathematical functionality -->

File: ros2_ws/src/xe_tham_do/description/lidar.xacro (robot description, xacro)
@@ -1,19 +1,4 @@
 <?xml version="1.0"?>
 <robot xmlns:xacro="http://www.ros.org/wiki/xacro" >
-    <!--
-        File này định nghĩa cảm biến laser (LIDAR) trong mô hình robot dưới dạng URDF/xacro.
-        - Khối <joint> "laser_joint" liên kết cố định giữa thân xe (chassis) và khung cảm biến laser (laser_frame).
-        - Khối <link> "laser_frame" mô tả hình học, va chạm và khối lượng của cảm biến laser:
-            + Gồm 2 hình trụ để mô phỏng hình dáng vật lý.
-            + Sử dụng macro xacro:inertial_cylinder để khai báo khối lượng và quán tính.
-        - Khối <gazebo> cấu hình cảm biến laser trong mô phỏng Gazebo:
-            + Đặt vật liệu màu đen.
-            + Khai báo cảm biến kiểu "ray" với các tham số:
-                * Góc quét: -3.14 đến 3.14 (360 mẫu).
-                * Khoảng cách đo: 0.3m đến 12m.
-                * Tần số cập nhật: 10Hz.
-            + Plugin "laser_controller" xuất dữ liệu về ROS topic "scan" dưới dạng sensor_msgs/LaserScan, gắn với frame "laser_frame".
-        Có thể sử dụng file này để tích hợp cảm biến laser cho robot trong mô phỏng (Gazebo) và thực tế (ROS).
-    -->
     <joint name="laser_joint" type="fixed">
         <parent link="chassis"/>

File: ros2_ws/src/xe_tham_do/description/robot.urdf.xacro (robot description, xacro)
@@ -1,17 +1,4 @@
 <?xml version="1.0"?>
 <robot xmlns:xacro="http://www.ros.org/wiki/xacro" name="robot">
-    <!--
-        File này là file xacro chính để xây dựng mô hình robot, cho phép cấu hình linh hoạt các thành phần phần cứng cũng như chế độ điều khiển/mô phỏng.
-        - Tham số use_ros2_control: Nếu true sẽ sử dụng ROS2 Control, nếu false sẽ dùng Gazebo Control.
-        - Tham số sim_mode: Chế độ mô phỏng (chưa sử dụng trong file này, có thể dùng cho các mục đích mở rộng).
-        - Bao gồm các file con:
-            + robot_core.xacro: Phần lõi, khung sườn và các link chính của robot.
-            + ros2_control.xacro: Cấu hình cho ROS2 Control (chỉ dùng khi use_ros2_control=true).
-            + gazebo_control.xacro: Cấu hình cho điều khiển trong Gazebo (chỉ dùng khi use_ros2_control=false).
-            + lidar.xacro: Định nghĩa cảm biến LIDAR cho robot.
-            + camera.xacro: Định nghĩa cảm biến camera chính.
-            + face.xacro: Định nghĩa phần mặt robot
-        File này giúp quản lý và cấu trúc các thành phần của robot một cách linh hoạt, dễ dàng chuyển đổi giữa mô phỏng và thực tế hoặc thêm bớt cảm biến.
-    -->
     <xacro:arg name="use_ros2_control" default="true"/>
     <xacro:arg name="sim_mode" default="false"/>

File: ros2_ws/src/xe_tham_do/description/robot_core.xacro (robot description, xacro)
@@ -1,19 +1,4 @@
 <?xml version="1.0"?>
 <robot xmlns:xacro="http://www.ros.org/wiki/xacro" >
-    <!--
-        File này định nghĩa mô hình cơ bản của robot di động sử dụng xacro/URDF.
-        - Bao gồm các thuộc tính hình học và vật lý cho chassis (thân xe), hai bánh xe chủ động (trái, phải) và một bánh tự do (caster wheel).
-        - Sử dụng các macro inertial từ file inertial_macros.xacro để tính toán quán tính cho các link.
-        - Các tham số (property) như kích thước, khối lượng của chassis, bánh xe... được khai báo rõ ràng đầu file, giúp dễ chỉnh sửa/tái sử dụng.
-        - Mỗi link đều có phần visual (hình dáng hiển thị), collision (hình học va chạm) và inertial (khối lượng/quán tính).
-        - Các khối <gazebo> giúp cấu hình vật liệu và thông số vật lý dùng khi mô phỏng trong Gazebo.
-        - Hệ thống joint gồm:
-            + base_footprint_joint: nối base_link với base_footprint.
-            + chassis_joint: nối base_link với chassis (thân xe).
-            + left_wheel_joint, right_wheel_joint: nối base_link với hai bánh xe, kiểu continuous để quay được.
-            + caster_wheel_joint: nối chassis với bánh tự do phía trước.
-        - Các màu sắc (material) được định nghĩa sẵn để tuỳ biến giao diện robot.
-        File này là nền tảng để tiếp tục mở rộng, lắp ráp thêm các cảm biến hoặc module khác cho robot di động.
-    -->
     <xacro:include filename="inertial_macros.xacro"/>
     <xacro:property name="chassis_length" value="0.45"/>

File: ros2_ws/src/xe_tham_do/description/ros2_control.xacro (robot description, xacro)
@@ -1,17 +1,4 @@
 <?xml version="1.0"?>
 <robot xmlns:xacro="http://www.ros.org/wiki/xacro">
-    <!--
-        File này định nghĩa cấu hình ros2_control cho robot, cho phép chuyển đổi linh hoạt giữa chế độ thực tế (RealRobot) và mô phỏng (Gazebo).
-        - Nếu không ở chế độ mô phỏng (sim_mode = false), sử dụng phần cứng thực DiffDriveArduino:
-            + Plugin: diffdrive_arduino/DiffDriveArduinoHardware
-            + Kết nối qua cổng serial, tốc độ baud và các thông số encoder.
-            + Các joint (left_wheel_joint, right_wheel_joint) khai báo interface điều khiển vận tốc và trạng thái.
-            + Tham số "enc_counts_per_rev": số xung encoder trên mỗi vòng của bánh xe.
-        - Nếu ở chế độ mô phỏng (sim_mode = true), sử dụng plugin mặc định của Gazebo:
-            + Plugin: gazebo_ros2_control/GazeboSystem
-            + Cấu hình interface cho các joint giống như thực tế.
-        - Phần <gazebo> cuối file khai báo plugin gazebo_ros2_control, chỉ định các file cấu hình controller cho ROS2 và Gazebo.
-        File này giúp dễ dàng chuyển đổi giữa điều khiển thực tế và mô phỏng chỉ với một biến sim_mode.
-    -->
     <xacro:unless value="$(arg sim_mode)">
         <ros2_control name="RealRobot" type="system">
