Commit message: add

File: ros2_ws/src/xe_tham_do/description/lidar.xacro (robot description, xacro)
@@ -4,34 +4,27 @@
         <parent link="chassis"/>
         <child link="laser_frame"/>
-        <origin xyz="0.122 0 0.212" rpy="0 0 0"/>
+        <origin  xyz="0.28 0 0.1405 " rpy="0 0 0"/>
     </joint>
     <link name="laser_frame">
         <visual>
             <geometry>
-                <cylinder radius="0.05" length="0.04"/>
+                <cylinder length="0.03" radius="0.052" />
             </geometry>
-            <material name="black"/>
-        </visual>
-        <visual>
-            <origin xyz="0 0 -0.05"/>
-            <geometry>
-                <cylinder radius="0.01" length="0.1"/>
-            </geometry>
-            <material name="black"/>
+                <material name="red" />
         </visual>
         <collision>
             <geometry>
-                <cylinder radius="0.05" length="0.04"/>
+                <cylinder length="0.03" radius="0.052" />
             </geometry>
         </collision>
-        <xacro:inertial_cylinder mass="0.1" length="0.04" radius="0.05">
-            <origin xyz="0 0 0" rpy="0 0 0"/>
+        <xacro:inertial_cylinder mass="0.1" length="0.03" radius="0.052">
+            <origin xyz="0 0 0" rpy="0 0 0" />
         </xacro:inertial_cylinder>
     </link>
     <gazebo reference="laser_frame">
-        <material>Gazebo/Black</material>
+        <material>Gazebo/Red</material>
         <sensor name="laser" type="ray">
             <pose> 0 0 0 0 0 0 </pose>
-            <visualize>false</visualize>
+            <visualize>true</visualize>
             <update_rate>10</update_rate>
             <ray>

Commit message: add

File: ros2_ws/src/xe_tham_do/description/lidar.xacro (robot description, xacro)
@@ -4,20 +4,20 @@
         <parent link="chassis"/>
         <child link="laser_frame"/>
-        <origin  xyz="0.28 0 0.1405 " rpy="0 0 0"/>
+        <origin xyz="0.122 0 0.212" rpy="0 0 0"/>
     </joint>
     <link name="laser_frame">
         <visual>
             <geometry>
-                <cylinder length="0.03" radius="0.052" />
+                <cylinder radius="0.05" length="0.04"/>
             </geometry>
-                <material name="red" />
+            <material name="black"/>
         </visual>
         <collision>
             <geometry>
-                <cylinder length="0.03" radius="0.052" />
+                <cylinder radius="0.05" length="0.04"/>
             </geometry>
         </collision>
         <xacro:inertial_cylinder mass="0.1" length="0.03" radius="0.052">
-            <origin xyz="0 0 0" rpy="0 0 0" />
+            <origin xyz="0 0 0" rpy="0 0 0"/>
         </xacro:inertial_cylinder>
     </link>

File: ros2_ws/src/xe_tham_do/description/robot_core.xacro (robot description, xacro)
@@ -9,5 +9,5 @@
     <xacro:property name="wheel_thickness" value="0.01"/>
     <xacro:property name="wheel_mass" value="0.1"/>
-    <xacro:property name="wheel_offset_x" value="0.226"/>
+    <xacro:property name="wheel_offset_x" value="0.05"/>
     <xacro:property name="wheel_offset_y" value="0.14"/>
     <xacro:property name="wheel_offset_z" value="0.01"/>

Commit message: add

File: ros2_ws/src/xe_tham_do/description/lidar.xacro (robot description, xacro)
@@ -4,5 +4,5 @@
         <parent link="chassis"/>
         <child link="laser_frame"/>
-        <origin xyz="0.122 0 0.212" rpy="0 0 0"/>
+        <origin xyz="0.14 0 0.25" rpy="0 0 0"/>
     </joint>
     <link name="laser_frame">

Commit message: add

File: ros2_ws/src/xe_tham_do/description/lidar.xacro (robot description, xacro)
@@ -4,5 +4,5 @@
         <parent link="chassis"/>
         <child link="laser_frame"/>
-        <origin xyz="0.14 0 0.25" rpy="0 0 0"/>
+        <origin xyz="0.26 0 0.25" rpy="0 0 0"/>
     </joint>
     <link name="laser_frame">

Commit message: add

File: ros2_ws/src/xe_tham_do/description/lidar.xacro (robot description, xacro)
@@ -4,5 +4,5 @@
         <parent link="chassis"/>
         <child link="laser_frame"/>
-        <origin xyz="0.26 0 0.25" rpy="0 0 0"/>
+        <origin xyz="0.26 0 0.212" rpy="0 0 0"/>
     </joint>
     <link name="laser_frame">
@@ -13,4 +13,11 @@
             <material name="black"/>
         </visual>
+        <visual>
+            <origin xyz="0 0 -0.05"/>
+            <geometry>
+                <cylinder radius="0.01" length="0.1"/>
+            </geometry>
+            <material name="black"/>
+        </visual>
         <collision>
             <geometry>
@@ -18,13 +25,13 @@
             </geometry>
         </collision>
-        <xacro:inertial_cylinder mass="0.1" length="0.03" radius="0.052">
+        <xacro:inertial_cylinder mass="0.1" length="0.04" radius="0.05">
             <origin xyz="0 0 0" rpy="0 0 0"/>
         </xacro:inertial_cylinder>
     </link>
     <gazebo reference="laser_frame">
-        <material>Gazebo/Red</material>
+        <material>Gazebo/Black</material>
         <sensor name="laser" type="ray">
             <pose> 0 0 0 0 0 0 </pose>
-            <visualize>true</visualize>
+            <visualize>false</visualize>
             <update_rate>10</update_rate>
             <ray>

File: ros2_ws/src/xe_tham_do/description/robot_core.xacro (robot description, xacro)
@@ -2,17 +2,17 @@
 <robot xmlns:xacro="http://www.ros.org/wiki/xacro" >
     <xacro:include filename="inertial_macros.xacro"/>
-    <xacro:property name="chassis_length" value="0.4"/>
-    <xacro:property name="chassis_width" value="0.26"/>
-    <xacro:property name="chassis_height" value="0.15"/>
+    <xacro:property name="chassis_length" value="0.49"/>
+    <xacro:property name="chassis_width" value="0.28"/>
+    <xacro:property name="chassis_height" value="0.13"/>
     <xacro:property name="chassis_mass" value="5.0"/>
-    <xacro:property name="wheel_radius" value="0.032"/>
-    <xacro:property name="wheel_thickness" value="0.011"/>
-    <xacro:property name="wheel_mass" value="0.1"/>
-    <xacro:property name="wheel_offset_x" value="0.38"/>
-    <xacro:property name="wheel_offset_y" value="0.135"/>
+    <xacro:property name="wheel_radius" value="0.034"/>
+    <xacro:property name="wheel_thickness" value="0.03"/>
+    <xacro:property name="wheel_mass" value="0.05"/>
+    <xacro:property name="wheel_offset_x" value="0.39"/>
+    <xacro:property name="wheel_offset_y" value="0.165"/>
     <xacro:property name="wheel_offset_z" value="0.01"/>
-    <xacro:property name="caster_wheel_radius" value="0.02"/>
+    <xacro:property name="caster_wheel_radius" value="0.015"/>
     <xacro:property name="caster_wheel_mass" value="0.01"/>
-    <xacro:property name="caster_wheel_offset_x" value="0"/>
+    <xacro:property name="caster_wheel_offset_x" value="0.075"/>
     <xacro:property name="caster_wheel_offset_z" value="${wheel_offset_z - wheel_radius + caster_wheel_radius}"/>
     <material name="white">
