Commit message: add

File: ros2_ws/src/xe_tham_do/description/robot_core.xacro (robot description, xacro)
@@ -17,8 +17,8 @@
     -->
     <xacro:include filename="inertial_macros.xacro"/>
-    <xacro:property name="chassis_length" value="0.335"/>
-    <xacro:property name="chassis_width" value="0.265"/>
-    <xacro:property name="chassis_height" value="0.138"/>
-    <xacro:property name="chassis_mass" value="1.0"/>
+    <xacro:property name="chassis_length" value="0.45"/>
+    <xacro:property name="chassis_width" value="0.3"/>
+    <xacro:property name="chassis_height" value="0.18"/>
+    <xacro:property name="chassis_mass" value="5.0"/>
     <xacro:property name="wheel_radius" value="0.065"/>
     <xacro:property name="wheel_thickness" value="0.01"/>
@@ -27,7 +27,7 @@
     <xacro:property name="wheel_offset_y" value="0.14"/>
     <xacro:property name="wheel_offset_z" value="0.01"/>
-    <xacro:property name="caster_wheel_radius" value="0.01"/>
+    <xacro:property name="caster_wheel_radius" value="0.03"/>
     <xacro:property name="caster_wheel_mass" value="0.01"/>
-    <xacro:property name="caster_wheel_offset_x" value="0.075"/>
+    <xacro:property name="caster_wheel_offset_x" value="0.38"/>
     <xacro:property name="caster_wheel_offset_z" value="${wheel_offset_z - wheel_radius + caster_wheel_radius}"/>
     <material name="white">

Commit message: add

File: ros2_ws/src/xe_tham_do/description/robot_core.xacro (robot description, xacro)
@@ -6,8 +6,8 @@
     <xacro:property name="chassis_height" value="0.18"/>
     <xacro:property name="chassis_mass" value="5.0"/>
-    <xacro:property name="wheel_radius" value="0.065"/>
+    <xacro:property name="wheel_radius" value="0.0325"/>
     <xacro:property name="wheel_thickness" value="0.01"/>
     <xacro:property name="wheel_mass" value="0.1"/>
-    <xacro:property name="wheel_offset_x" value="0.05"/>
+    <xacro:property name="wheel_offset_x" value="0.045"/>
     <xacro:property name="wheel_offset_y" value="0.14"/>
     <xacro:property name="wheel_offset_z" value="0.01"/>

Commit message: add

File: ros2_ws/src/xe_tham_do/description/robot_core.xacro (robot description, xacro)
@@ -9,5 +9,5 @@
     <xacro:property name="wheel_thickness" value="0.01"/>
     <xacro:property name="wheel_mass" value="0.1"/>
-    <xacro:property name="wheel_offset_x" value="0.045"/>
+    <xacro:property name="wheel_offset_x" value="0.226"/>
     <xacro:property name="wheel_offset_y" value="0.14"/>
     <xacro:property name="wheel_offset_z" value="0.01"/>

Commit message: add

File: ros2_ws/src/xe_tham_do/description/robot_core.xacro (robot description, xacro)
@@ -9,5 +9,5 @@
     <xacro:property name="wheel_thickness" value="0.01"/>
     <xacro:property name="wheel_mass" value="0.1"/>
-    <xacro:property name="wheel_offset_x" value="0.226"/>
+    <xacro:property name="wheel_offset_x" value="0"/>
     <xacro:property name="wheel_offset_y" value="0.14"/>
     <xacro:property name="wheel_offset_z" value="0.01"/>

Commit message: add

File: ros2_ws/src/xe_tham_do/description/robot_core.xacro (robot description, xacro)
@@ -9,10 +9,10 @@
     <xacro:property name="wheel_thickness" value="0.01"/>
     <xacro:property name="wheel_mass" value="0.1"/>
-    <xacro:property name="wheel_offset_x" value="0"/>
+    <xacro:property name="wheel_offset_x" value="0.38"/>
     <xacro:property name="wheel_offset_y" value="0.14"/>
     <xacro:property name="wheel_offset_z" value="0.01"/>
     <xacro:property name="caster_wheel_radius" value="0.03"/>
     <xacro:property name="caster_wheel_mass" value="0.01"/>
-    <xacro:property name="caster_wheel_offset_x" value="0.38"/>
+    <xacro:property name="caster_wheel_offset_x" value="0"/>
     <xacro:property name="caster_wheel_offset_z" value="${wheel_offset_z - wheel_radius + caster_wheel_radius}"/>
     <material name="white">

Commit message: add

File: ros2_ws/src/xe_tham_do/description/robot_core.xacro (robot description, xacro)
@@ -2,7 +2,7 @@
 <robot xmlns:xacro="http://www.ros.org/wiki/xacro" >
     <xacro:include filename="inertial_macros.xacro"/>
-    <xacro:property name="chassis_length" value="0.45"/>
-    <xacro:property name="chassis_width" value="0.3"/>
-    <xacro:property name="chassis_height" value="0.18"/>
+    <xacro:property name="chassis_length" value="0.4"/>
+    <xacro:property name="chassis_width" value="0.26"/>
+    <xacro:property name="chassis_height" value="0.15"/>
     <xacro:property name="chassis_mass" value="5.0"/>
     <xacro:property name="wheel_radius" value="0.0325"/>
@@ -10,5 +10,5 @@
     <xacro:property name="wheel_mass" value="0.1"/>
     <xacro:property name="wheel_offset_x" value="0.38"/>
-    <xacro:property name="wheel_offset_y" value="0.14"/>
+    <xacro:property name="wheel_offset_y" value="0.135"/>
     <xacro:property name="wheel_offset_z" value="0.01"/>
     <xacro:property name="caster_wheel_radius" value="0.03"/>

Commit message: add

File: ros2_ws/src/xe_tham_do/description/robot_core.xacro (robot description, xacro)
@@ -6,5 +6,5 @@
     <xacro:property name="chassis_height" value="0.15"/>
     <xacro:property name="chassis_mass" value="5.0"/>
-    <xacro:property name="wheel_radius" value="0.0325"/>
+    <xacro:property name="wheel_radius" value="0.032"/>
     <xacro:property name="wheel_thickness" value="0.01"/>
     <xacro:property name="wheel_mass" value="0.1"/>

Commit message: add

File: ros2_ws/src/xe_tham_do/description/robot_core.xacro (robot description, xacro)
@@ -7,10 +7,10 @@
     <xacro:property name="chassis_mass" value="5.0"/>
     <xacro:property name="wheel_radius" value="0.032"/>
-    <xacro:property name="wheel_thickness" value="0.01"/>
+    <xacro:property name="wheel_thickness" value="0.011"/>
     <xacro:property name="wheel_mass" value="0.1"/>
     <xacro:property name="wheel_offset_x" value="0.38"/>
     <xacro:property name="wheel_offset_y" value="0.135"/>
     <xacro:property name="wheel_offset_z" value="0.01"/>
-    <xacro:property name="caster_wheel_radius" value="0.03"/>
+    <xacro:property name="caster_wheel_radius" value="0.02"/>
     <xacro:property name="caster_wheel_mass" value="0.01"/>
     <xacro:property name="caster_wheel_offset_x" value="0"/>

Commit message: add

File: ros2_ws/src/xe_tham_do/description/robot_core.xacro (robot description, xacro)
@@ -2,13 +2,13 @@
 <robot xmlns:xacro="http://www.ros.org/wiki/xacro" >
     <xacro:include filename="inertial_macros.xacro"/>
-    <xacro:property name="chassis_length" value="0.49"/>
-    <xacro:property name="chassis_width" value="0.28"/>
-    <xacro:property name="chassis_height" value="0.13"/>
+    <xacro:property name="chassis_length" value="0.4"/>
+    <xacro:property name="chassis_width" value="0.26"/>
+    <xacro:property name="chassis_height" value="0.15"/>
     <xacro:property name="chassis_mass" value="5.0"/>
-    <xacro:property name="wheel_radius" value="0.034"/>
-    <xacro:property name="wheel_thickness" value="0.03"/>
+    <xacro:property name="wheel_radius" value="0.032"/>
+    <xacro:property name="wheel_thickness" value="0.02"/>
     <xacro:property name="wheel_mass" value="0.05"/>
     <xacro:property name="wheel_offset_x" value="0.39"/>
-    <xacro:property name="wheel_offset_y" value="0.165"/>
+    <xacro:property name="wheel_offset_y" value="0.1425"/>
     <xacro:property name="wheel_offset_z" value="0.01"/>
     <xacro:property name="caster_wheel_radius" value="0.015"/>
